File: poc-one/analog.kicad_sch (KiCad schematic)
At the start: 16 parts, among them J2 TOUCH_FANOUT, Q7 XYC-PT0805BC-L4-D, U22 LMV321IDBVR

Commit message: fixed a couple resistors, reworked footprints incl. datasheets
Parts:
- J2: now left out of the parts list
Changed lines of the file:
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@@
 		(body_style 1)
 		(exclude_from_sim no)
-		(in_bom yes)
+		(in_bom no)
 		(on_board yes)
-		(in_pos_files yes)
+		(in_pos_files no)
 		(dnp no)
 		(fields_autoplaced yes)

Commit message: poc-one routed & schematic changes
Parts:
- TP10, TP11: now left out of the parts list
- renumbered C38 to C37, C37 to C38, J2 to J4, R46 to R42, R42 to R44, R44 to R46
Connections:
- net +3V3: no longer C36.2, C38.1, J4.11 (Pin_11), J4.13 (Pin_13), J4.3 (Pin_3), J4.5 (Pin_5), J4.7 (Pin_7), J4.9 (Pin_9), MK1.2 (GND), MK1.3 (GND), R42.2, R43.1, U22.2 (GND)
- new net GND: C36.2, C38.1, J4.11 (Pin_11), J4.13 (Pin_13), J4.3 (Pin_3), J4.5 (Pin_5), J4.7 (Pin_7), J4.9 (Pin_9), MK1.2 (GND), MK1.3 (GND), R42.2, R43.1, U22.2 (GND)
