File: poc-one/led_control.kicad_sch (KiCad schematic)
At the start: 38 parts, among them Q1 SS8550 Y2 200-350, Q2 SS8550 Y2 200-350, Q3 SS8550 Y2 200-350, Q5 SS8550 Y2 200-350, U10 74HC595D, U11 74HC595D, U12 74HC595D, U13 74HC595D, U14 74HC595D, U15 74HC595D, U16 74HC595D, U17 74HC595D, U18 74HC595D, U19 74HC595D, U20 74HC595D, U4 74HC138, U5 74HC138, U6 74HC138, U7 74HC138, U8 74HC138, U9 74HC595D

Commit message: schematic-v2
Parts:
- added C24, C28, C29, C30, C31, C32, C33, C34: C_Polarized, Capacitor_SMD:CP_Elec_5x5.4, symbol Device:C_Polarized
- added R39: 10, symbol Device:R
- added TP8: DISPLAY_SENSE-, symbol Connector:TestPoint
- added TP9: DISPLAY_SENSE+, symbol Connector:TestPoint
Connections:
- net +3V3: now also U6.16 (VCC), U7.16 (VCC), U8.16 (VCC), U8.4 (~{E0}), U8.5 (~{E1}), R39.1, TP9.1; no longer Q1.2 (E), Q2.2 (E), Q3.2 (E), Q5.2 (E)
- net GND: now also U6.6 (E2), U6.8 (GND), U7.6 (E2), U7.8 (GND), U8.6 (E2), U8.8 (GND), C24.2, C28.2, C29.2, C30.2, C31.2, C32.2, C33.2, C34.2
- net at U6.4 (~{E0}), U8.13 (~{Y2}): now also U6.5 (~{E1})
- net at U7.4 (~{E0}), U8.12 (~{Y3}): now also U7.5 (~{E1})
- new net: C24.1, C28.1, C29.1, C30.1, C31.1, C32.1, C33.1, C34.1, Q1.2 (E), Q2.2 (E), Q3.2 (E), Q5.2 (E), R39.2, TP8.1
- no-connect marks 32 -> 200
Other:
- sheet LED_matrix: file leds.kicad_sch -> led_matrix.kicad_sch
- note added: "PNP gain ~40-120 max LED array current ~576mA per row => ~15mA max on the PNP base => 220Ω @ 3.3V"
- moved on the sheet: U10, U12, U15, U16, U17, U18, U19, U20

Commit message: poc-one update & bom
Parts:
- C24, C28, C29, C30, C31, C32, C33, C34: value C_Polarized -> 100u
- R39: footprint (none) -> Resistor_SMD:R_0402_1005Metric
- TP8, TP9: footprint (none) -> TestPoint:TestPoint_Pad_D1.5mm
Changed lines of the file:
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@@
 	)
 	(junction
-		(at 175.26 171.45)
+		(at 213.36 179.07)
 		(diameter 0)
 		(color 0 0 0 0)
 	)
 	(junction
-		(at 213.36 179.07)
+		(at 205.74 179.07)
 		(diameter 0)
 		(color 0 0 0 0)
 	)
 	(junction
-		(at 205.74 179.07)
+		(at 175.26 179.07)
 		(diameter 0)
 		(color 0 0 0 0)
@@
 	)
 	(junction
-		(at 175.26 179.07)
-		(diameter 0)
-		(color 0 0 0 0)
-	)
-	(junction
 		(at 190.5 179.07)
 		(diameter 0)
@@
 	)
 	(junction
+		(at 175.26 171.45)
+		(diameter 0)
+		(color 0 0 0 0)
+	)
+	(junction
 		(at 355.6 87.63)
 		(diameter 0)
@@
 		(exclude_from_sim no)
 		(in_bom yes)
-		(on_board yes)
+		(on_board no)
 		(in_pos_files yes)
 		(dnp yes)
@@
 			)
 		)
-		(property "Value" "C_Polarized"
+		(property "Value" "100u"
 			(at 186.69 175.6409 0)
 			(show_name no)
@@
 		(exclude_from_sim no)
 		(in_bom yes)
-		(on_board yes)
+		(on_board no)
 		(in_pos_files yes)
 		(dnp yes)
@@
 			)
 		)
-		(property "Value" "C_Polarized"
+		(property "Value" "100u"
 			(at 201.93 175.6409 0)
 			(show_name no)
@@
 		(exclude_from_sim no)
 		(in_bom yes)
-		(on_board yes)
+		(on_board no)
 		(in_pos_files yes)
 		(dnp yes)
@@
 			)
 		)
-		(property "Value" "C_Polarized"
+		(property "Value" "100u"
 			(at 217.17 175.6409 0)
 			(show_name no)
@@
 		(exclude_from_sim no)
 		(in_bom yes)
-		(on_board yes)
+		(on_board no)
 		(in_pos_files yes)
 		(dnp yes)
@@
 			)
 		)
-		(property "Value" "C_Polarized"
+		(property "Value" "100u"
 			(at 224.79 175.6409 0)
 			(show_name no)
@@
 			)
 		)
-		(property "Value" "C_Polarized"
+		(property "Value" "100u"
 			(at 179.07 175.6409 0)
 			(show_name no)
@@
 		(exclude_from_sim no)
 		(in_bom yes)
-		(on_board yes)
+		(on_board no)
 		(in_pos_files yes)
 		(dnp yes)
@@
 			)
 		)
-		(property "Value" "C_Polarized"
+		(property "Value" "100u"
 			(at 194.31 175.6409 0)
 			(show_name no)
@@
 		(exclude_from_sim no)
 		(in_bom yes)
-		(on_board yes)
+		(on_board no)
 		(in_pos_files yes)
 		(dnp yes)
@@
 			)
 		)
-		(property "Value" "C_Polarized"
+		(property "Value" "100u"
 			(at 209.55 175.6409 0)
 			(show_name no)
@@
 			)
 		)
-		(property "Footprint" ""
+		(property "Footprint" "TestPoint:TestPoint_Pad_D1.5mm"
 			(at 171.45 167.64 0)
 			(hide yes)
@@
 			)
 		)
-		(property "Footprint" ""
+		(property "Footprint" "Resistor_SMD:R_0402_1005Metric"
 			(at 160.02 170.688 90)
 			(hide yes)
@@
 		(exclude_from_sim no)
 		(in_bom yes)
-		(on_board yes)
+		(on_board no)
 		(in_pos_files yes)
 		(dnp yes)
@@
 			)
 		)
-		(property "Value" "C_Polarized"
+		(property "Value" "100u"
 			(at 232.41 175.6409 0)
 			(show_name no)
@@
 			)
 		)
-		(property "Footprint" ""
+		(property "Footprint" "TestPoint:TestPoint_Pad_D1.5mm"
 			(at 157.48 168.91 0)
 			(hide yes)

Commit message: poc-one routed & schematic changes
Parts:
- R23: value 0 -> 10k
- TP8: renamed from TP9; now left out of the parts list
- TP9: renamed from TP8; now left out of the parts list
- U11: renamed from U10; now left out of the parts list
- U13: renamed from U12; now left out of the parts list
- U15: renamed from U14; now left out of the parts list
- U16: renamed from U15; now left out of the parts list
- U17: renamed from U16; now left out of the parts list
- U18: renamed from U17; now left out of the parts list
- U19: renamed from U18; now left out of the parts list
- U20: renamed from U19; now left out of the parts list
- U21: renamed from U20; now left out of the parts list
- U5: renamed from U8; now left out of the parts list
- U7: renamed from U5; now left out of the parts list
- U8: renamed from U6; now left out of the parts list
- U9: renamed from U7; now left out of the parts list
- renumbered C24 to C27, Q5 to Q3, Q1 to Q4, Q2 to Q5, Q3 to Q6, R39 to R25, R25 to R26, R26 to R27, R27 to R28, R28 to R29, R29 to R30, R12 to R31, R30 to R32, R13 to R33, R15 to R34, R31 to R35, R16 to R36, R18 to R37, R19 to R38, R21 to R39, R22 to R40, U9 to U10, U11 to U12, U13 to U14, U4 to U6
