File: poc-one/leds.kicad_sch (KiCad schematic)
At the start: 16 parts

Commit message: poc-one routed & schematic changes
Parts:
- renumbered D4 to D1, D13 to D10, D14 to D11, D15 to D12, D16 to D13, D17 to D14, D18 to D15, D19 to D16, D5 to D2, D6 to D3, D7 to D4, D8 to D5, D9 to D6, D10 to D7, D11 to D8, D12 to D9
Connections:
- no-connect marks 114 -> 0
