File: hardware/full-poc/battery.kicad_sch (KiCad schematic)
At the start: 31 parts, among them J3 Connector, USB-TYPE-C-16P, Q22 BC857BS, Q23 SI2302, SW3 BAT_SOFT_OFF HY-DSIC02LS, U19 H7650-33PR, U24 BQ24195LRGER

Commit message: full board + panel
Parts:
- renumbered BT1 to BT301, C57 to C301, C61 to C302, C62 to C303, C58 to C304, C60 to C305, C63 to C306, C64 to C307, C59 to C308, J3 to J301, L2 to L301, Q22 to Q301, Q23 to Q302, R56 to R301, R55 to R302, R59 to R303, R63 to R304, R62 to R305, R64 to R306, R60 to R307, R61 to R308, R66 to R309, R65 to R310, SW3 to SW301, TP18 to TP301, TP12 to TP302, TP17 to TP303, TP13 to TP304, TP14 to TP305, U24 to U301, U19 to U302
