File: hardware/full-poc/display_unit.kicad_sch (KiCad schematic)
At the start: 39 parts, among them J5 DEBUG, J7 Connector, USB-TYPE-C-16P, Q21 XYC-PT0805BC-L4-D, SW4 KH-6X6X5H-STM, SW7 KH-6X6X5H-STM, U30 RP2354_80QFN, Y1 ABM8-272-T3

Commit message: full board + panel
Parts:
- renumbered C6 to C201, C8 to C202, C9 to C203, C10 to C204, C12 to C205, C13 to C206, C14 to C207, C15 to C208, C16 to C209, C17 to C210, C18 to C211, C39 to C212, C11 to C213, C7 to C214, C4 to C215, C5 to C216, C1 to C217, C2 to C218, J5 to J201, J7 to J202, L1 to L201, Q21 to Q201, R5 to R201, R7 to R202, R8 to R203, R3 to R204, R2 to R205, R54 to R206, R53 to R207, R42 to R208, SW7 to SW201, SW4 to SW202, TP16 to TP201, TP1 to TP202, TP2 to TP203, TP3 to TP204, TP4 to TP205, U30 to U201, Y1 to Y201
