File: hardware/full-poc/led_control.kicad_sch (KiCad schematic)
At the start: 183 parts, among them Q1 BC857BS, Q10 BC857BS, Q11 BC857BS, Q12 BC857BS, Q13 BC857BS, Q14 BC857BS, Q15 BC857BS, Q16 BC857BS, Q17 BC857BS, Q18 BC857BS, Q19 BC857BS, Q2 BC857BS, Q20 BC857BS, Q3 BC857BS, Q4 BC857BS, Q5 BC857BS, Q6 BC857BS, Q7 BC857BS, Q8 BC857BS, Q9 BC857BS, U1 74HC595BQ, U10 74HC595BQ, U11 74HC595BQ, U12 74HC595BQ, U13 74HC138LQ/TR, U14 74HC138LQ/TR, U15 74HC138LQ/TR, U16 74HC138LQ/TR, U17 74HC138LQ/TR, U18 74HC138LQ/TR, U2 74HC595BQ, U3 74HC595BQ, U4 74HC595BQ, U5 74HC595BQ, U6 74HC595BQ, U7 74HC595BQ, U8 74HC595BQ, U9 74HC595BQ

Commit message: full board + panel
Parts:
- renumbered C26 to C401, C27 to C402, C28 to C403, C29 to C404, C30 to C405, C31 to C406, C32 to C407, C33 to C408, C34 to C409, Q1 to Q401, Q2 to Q402, Q3 to Q403, Q4 to Q404, Q5 to Q405, Q6 to Q406, Q7 to Q407, Q8 to Q408, Q9 to Q409, Q10 to Q410, Q11 to Q411, Q12 to Q412, Q13 to Q413, Q14 to Q414, Q15 to Q415, Q16 to Q416, Q17 to Q417, Q18 to Q418, Q19 to Q419, Q20 to Q420, R67 to R401, R68 to R402, R69 to R403, R70 to R404, R71 to R405, R72 to R406, R73 to R407, R74 to R408, R80 to R409, R75 to R410, R78 to R411, R81 to R412, R76 to R413, R79 to R414, R82 to R415, R77 to R416, R86 to R417, R89 to R418, R84 to R419, R87 to R420, R90 to R421, R85 to R422, R88 to R423, R83 to R424, R91 to R425, R99 to R426, R107 to R427, R92 to R428, R100 to R429, R108 to R430, R93 to R431, R101 to R432, R109 to R433, R94 to R434, R102 to R435, R110 to R436, R95 to R437, R103 to R438, R111 to R439, R96 to R440, R104 to R441, R112 to R442, R97 to R443, R105 to R444, R113 to R445, R98 to R446, R106 to R447, R114 to R448, R115 to R449, R123 to R450, R131 to R451, R116 to R452, R124 to R453, R132 to R454, R117 to R455, R125 to R456, R133 to R457, R118 to R458, R126 to R459, R134 to R460, R119 to R461, R127 to R462, R135 to R463, R120 to R464, R128 to R465, R136 to R466, R121 to R467, R129 to R468, R137 to R469, R122 to R470, R130 to R471, R138 to R472, R139 to R473, R147 to R474, R155 to R475, R140 to R476, R148 to R477, R156 to R478, R141 to R479, R149 to R480, R157 to R481, R142 to R482, R150 to R483, R158 to R484, R143 to R485, R151 to R486, R159 to R487, R144 to R488, R152 to R489, R160 to R490, R145 to R491, R153 to R492, R161 to R493, R146 to R494, R154 to R495, R162 to R496, R24 to R497, R26 to R498, R27 to R499, R28 to R500, R25 to R501, R29 to R502, R30 to R503, R31 to R504, R32 to R505, R34 to R506, R36 to R507, R38 to R508, R33 to R509, R35 to R510, R37 to R511, R39 to R512, R40 to R513, R164 to R514, R166 to R515, R168 to R516, R163 to R517, R165 to R518, R167 to R519, R169 to R520, R170 to R521, R172 to R522, R174 to R523, R176 to R524, R171 to R525, R173 to R526, R175 to R527, R177 to R528, R178 to R529, R180 to R530, R182 to R531, R184 to R532, R179 to R533, R181 to R534, R183 to R535, R185 to R536, U1 to U401, U2 to U402, U3 to U403, U4 to U404, U5 to U405, U6 to U406, U7 to U407, U8 to U408, U9 to U409, U10 to U410, U11 to U411, U12 to U412, U14 to U413, U13 to U414, U15 to U415, U16 to U416, U17 to U417, U18 to U418
