File: hardware/full-poc/mcu.kicad_sch (KiCad schematic)
At the start: 36 parts, among them J1 SAO V1.69bis, J6 DEBUG, Q22 BC857BS, SW1 KH-6X6X5H-STM, SW2 KH-6X6X5H-STM, U23 RP2354_80QFN, Y2 ABM8-272-T3

Commit message: full board + panel
Parts:
- added CAP101: CAP1, symbol Connector:TestPoint_Flag
- added CAP102: CAP2, symbol Connector:TestPoint_Flag
- added CAP103: CAP3, symbol Connector:TestPoint_Flag
- added CAP104: CAP4, symbol Connector:TestPoint_Flag
- J102: renamed from J1; now left out of the parts list
- renumbered BZ1 to BZ101, C43 to C101, C45 to C102, C46 to C103, C47 to C104, C49 to C105, C50 to C106, C51 to C107, C52 to C108, C53 to C109, C54 to C110, C55 to C111, C56 to C112, C48 to C113, C44 to C114, C41 to C115, C42 to C116, C3 to C117, C40 to C118, J6 to J101, L3 to L101, Q22 to Q301, R50 to R101, R51 to R102, R52 to R103, R49 to R104, R41 to R105, R47 to R106, R48 to R107, SW1 to SW101, SW2 to SW102, TP19 to TP101, U23 to U101, Y2 to Y101
Connections:
- net at U101.49 (GPIO40_ADC0): now also CAP101.1
- net at U101.52 (GPIO41_ADC1): now also CAP102.1
- net at U101.53 (GPIO42_ADC2): now also CAP103.1
- net at U101.54 (GPIO43_ADC3): now also CAP104.1
- no-connect marks 40 -> 36
