File: hardware/full-poc/poc-full.kicad_pcb (KiCad board)
At the start: 4 copper layers, 190 x 80 mm, 1358 parts, among them J1 SAO V1.69bis, J3 Connector, USB-TYPE-C-16P, J5 DEBUG, J6 DEBUG, J7 Connector, USB-TYPE-C-16P, Q1 BC857BS, Q10 BC857BS, Q11 BC857BS, Q12 BC857BS, Q13 BC857BS, Q14 BC857BS, Q15 BC857BS, Q16 BC857BS, Q17 BC857BS, Q18 BC857BS, Q19 BC857BS, Q2 BC857BS, Q20 BC857BS, Q21 XYC-PT0805BC-L4-D, Q22 BC857BS, Q23 SI2302, Q3 BC857BS, Q4 BC857BS, Q5 BC857BS, Q6 BC857BS, Q7 BC857BS, Q8 BC857BS, Q9 BC857BS, SW1 KH-6X6X5H-STM, SW2 KH-6X6X5H-STM, SW3 BAT_SOFT_OFF HY-DSIC02LS, SW4 KH-6X6X5H-STM, SW7 KH-6X6X5H-STM, U1 74HC595BQ, U10 74HC595BQ, U11 74HC595BQ, U12 74HC595BQ, U13 74HC138LQ/TR, U14 74HC138LQ/TR, U15 74HC138LQ/TR, U16 74HC138LQ/TR, U17 74HC138LQ/TR, U18 74HC138LQ/TR, U19 H7650-33PR, U2 74HC595BQ, U20 CMT2219A, U21 ST25R3916B-AQWT, U23 RP2354_80QFN, U24 BQ24195LRGER, U3 74HC595BQ, U30 RP2354_80QFN, U4 74HC595BQ, U5 74HC595BQ, U6 74HC595BQ, U7 74HC595BQ, U8 74HC595BQ, U9 74HC595BQ, Y1 ABM8-272-T3, Y2 ABM8-272-T3, Y3 TAXM26M4RHBCCT2T, Y4 5YMA27120091KF50EB

Commit message: full board + panel
Parts:
- removed Q1, Q10, Q11, Q12, Q13, Q14, Q15, Q16, Q17, Q18, Q19, Q2, Q20, Q3, Q4, Q5, Q6, Q7, Q8, Q9: BC857BS, Package_TO_SOT_SMD:SOT-363_SC-70-6
- removed R100, R123, R124, R125, R126, R127, R128, R129, R130, R147, R148, R149, R150, R151, R152, R153, R154, R71, R74, R78, R79, R86, R87, R88, R99: 360, Resistor_SMD:R_0402_1005Metric
- removed the R101 at (240.2, 179.5)
- removed the R102 at (215.6, 287.1)
- removed the R103 at (215.6, 289.0)
- removed the R104 at (215.6, 291.0)
- removed the R105 at (215.6, 293.0)
- removed the R106 at (212.7, 267.1)
- removed the R107 at (237.2, 176.9)
- removed R108, R109, R110, R111, R112, R113, R114, R131, R132, R133, R134, R135, R136, R137, R138, R155, R156, R157, R158, R159, R160, R161, R162, R72, R80, R81, R82, R83, R89, R90: 82, Resistor_SMD:R_0402_1005Metric
- removed R115, R116, R117, R118, R119, R120, R121, R122, R139, R140, R141, R142, R143, R144, R145, R146, R70, R73, R75, R76, R77, R84, R85, R91, R92, R93, R94, R95, R96, R97, R98: 130, Resistor_SMD:R_0402_1005Metric
- removed R163, R164, R165, R166, R167, R168, R169, R170, R171, R172, R173, R174, R175, R176, R177, R178, R179, R180, R181, R182, R183, R184, R185, R24, R25, R26, R27, R28, R29, R30, R31, R32, R33, R34, R35, R36, R37, R38, R39, R40: 1k, Resistor_SMD:R_0402_1005Metric
- removed U10, U11, U12, U2, U3, U4, U5, U6, U7, U8, U9: 74HC595BQ, Package_DFN_QFN:DHVQFN-16-1EP_2.5x3.5mm_P0.5mm_EP1x2mm
- removed U13, U14, U15, U16, U17: 74HC138LQ/TR, Package_DFN_QFN:QFN-16-1EP_3x3mm_P0.5mm_EP1.7x1.7mm_ThermalVias
- added CAP101: CAP1, Connector_Wire:SolderWirePad_1x01_SMD_5x10mm, F.Cu at (315.6, 155.7)
- added CAP102: CAP2, Connector_Wire:SolderWirePad_1x01_SMD_5x10mm, F.Cu at (321.6, 155.7)
- added CAP103: CAP3, Connector_Wire:SolderWirePad_1x01_SMD_5x10mm, F.Cu at (327.6, 155.7)
- added CAP104: CAP4, Connector_Wire:SolderWirePad_1x01_SMD_5x10mm, F.Cu at (333.6, 155.7)
- added Q401: BC857BS, Package_TO_SOT_SMD:SOT-363_SC-70-6, B.Cu at (242.0, 162.4)
- added Q402: BC857BS, Package_TO_SOT_SMD:SOT-363_SC-70-6, B.Cu at (242.0, 165.9)
- added Q403: BC857BS, Package_TO_SOT_SMD:SOT-363_SC-70-6, B.Cu at (242.0, 169.4)
- added Q404: BC857BS, Package_TO_SOT_SMD:SOT-363_SC-70-6, B.Cu at (242.0, 172.9)
- added Q405: BC857BS, Package_TO_SOT_SMD:SOT-363_SC-70-6, B.Cu at (242.0, 176.4)
- added Q406: BC857BS, Package_TO_SOT_SMD:SOT-363_SC-70-6, B.Cu at (242.0, 179.9)
- added Q407: BC857BS, Package_TO_SOT_SMD:SOT-363_SC-70-6, B.Cu at (242.0, 183.4)
- added Q408: BC857BS, Package_TO_SOT_SMD:SOT-363_SC-70-6, B.Cu at (242.0, 186.9)
- added Q409: BC857BS, Package_TO_SOT_SMD:SOT-363_SC-70-6, B.Cu at (242.0, 190.4)
- added Q410: BC857BS, Package_TO_SOT_SMD:SOT-363_SC-70-6, B.Cu at (242.0, 193.9)
- added Q411: BC857BS, Package_TO_SOT_SMD:SOT-363_SC-70-6, B.Cu at (242.0, 197.4)
- added Q412: BC857BS, Package_TO_SOT_SMD:SOT-363_SC-70-6, B.Cu at (242.0, 200.9)
- added Q413: BC857BS, Package_TO_SOT_SMD:SOT-363_SC-70-6, B.Cu at (242.0, 204.4)
- added Q414: BC857BS, Package_TO_SOT_SMD:SOT-363_SC-70-6, B.Cu at (242.0, 207.9)
- added Q415: BC857BS, Package_TO_SOT_SMD:SOT-363_SC-70-6, B.Cu at (242.0, 211.4)
- added Q416: BC857BS, Package_TO_SOT_SMD:SOT-363_SC-70-6, B.Cu at (242.0, 214.9)
- added R401: 130, Resistor_SMD:R_0402_1005Metric, B.Cu at (230.6, 216.5)
- added R402: 360, Resistor_SMD:R_0402_1005Metric, B.Cu at (232.6, 216.0)
- added R403: 82, Resistor_SMD:R_0402_1005Metric, B.Cu at (230.6, 215.5)
- added R404: 130, Resistor_SMD:R_0402_1005Metric, B.Cu at (232.6, 215.0)
- added R405: 360, Resistor_SMD:R_0402_1005Metric, B.Cu at (230.6, 214.2)
- added R406: 82, Resistor_SMD:R_0402_1005Metric, B.Cu at (232.6, 213.7)
- added R407: 130, Resistor_SMD:R_0402_1005Metric, B.Cu at (230.6, 213.2)
- added R408: 360, Resistor_SMD:R_0402_1005Metric, B.Cu at (232.6, 212.7)
- added R409: 82, Resistor_SMD:R_0402_1005Metric, B.Cu at (230.6, 211.9)
- added R410: 130, Resistor_SMD:R_0402_1005Metric, B.Cu at (232.6, 211.4)
- added R411: 360, Resistor_SMD:R_0402_1005Metric, B.Cu at (230.6, 210.9)
- added R412: 82, Resistor_SMD:R_0402_1005Metric, B.Cu at (232.6, 210.4)
- added R413: 130, Resistor_SMD:R_0402_1005Metric, B.Cu at (230.6, 209.5)
- added R414: 360, Resistor_SMD:R_0402_1005Metric, B.Cu at (232.6, 209.0)
- added R415: 82, Resistor_SMD:R_0402_1005Metric, B.Cu at (230.6, 208.5)
- added R416: 130, Resistor_SMD:R_0402_1005Metric, B.Cu at (232.6, 208.0)
- added R417: 360, Resistor_SMD:R_0402_1005Metric, B.Cu at (230.6, 207.2)
- added R418: 82, Resistor_SMD:R_0402_1005Metric, B.Cu at (232.6, 206.7)
- added R419: 130, Resistor_SMD:R_0402_1005Metric, B.Cu at (230.6, 206.2)
- added R420: 360, Resistor_SMD:R_0402_1005Metric, B.Cu at (232.6, 205.7)
- added R421: 82, Resistor_SMD:R_0402_1005Metric, B.Cu at (230.6, 204.9)
- added R422: 130, Resistor_SMD:R_0402_1005Metric, B.Cu at (232.6, 204.4)
- added R423: 360, Resistor_SMD:R_0402_1005Metric, B.Cu at (230.6, 203.9)
- added R424: 82, Resistor_SMD:R_0402_1005Metric, B.Cu at (232.6, 203.4)
- added R425: 130, Resistor_SMD:R_0402_1005Metric, B.Cu at (230.6, 202.6)
- added R426: 360, Resistor_SMD:R_0402_1005Metric, B.Cu at (232.6, 202.1)
- added R427: 82, Resistor_SMD:R_0402_1005Metric, B.Cu at (230.6, 201.6)
- added R428: 130, Resistor_SMD:R_0402_1005Metric, B.Cu at (232.6, 201.1)
- added R429: 360, Resistor_SMD:R_0402_1005Metric, B.Cu at (230.6, 200.3)
- added R430: 82, Resistor_SMD:R_0402_1005Metric, B.Cu at (232.6, 199.8)
- added R431: 130, Resistor_SMD:R_0402_1005Metric, B.Cu at (230.6, 199.3)
- added R432: 360, Resistor_SMD:R_0402_1005Metric, B.Cu at (232.6, 198.8)
- added R433: 82, Resistor_SMD:R_0402_1005Metric, B.Cu at (230.6, 197.9)
- added R434: 130, Resistor_SMD:R_0402_1005Metric, B.Cu at (232.6, 197.4)
- added R435: 360, Resistor_SMD:R_0402_1005Metric, B.Cu at (230.6, 196.9)
- added R436: 82, Resistor_SMD:R_0402_1005Metric, B.Cu at (232.6, 196.4)
- added R437: 130, Resistor_SMD:R_0402_1005Metric, B.Cu at (230.6, 195.6)
- added R438: 360, Resistor_SMD:R_0402_1005Metric, B.Cu at (232.6, 195.1)
- added R439: 82, Resistor_SMD:R_0402_1005Metric, B.Cu at (230.6, 194.6)
- added R440: 130, Resistor_SMD:R_0402_1005Metric, B.Cu at (232.6, 194.1)
- added R441: 360, Resistor_SMD:R_0402_1005Metric, B.Cu at (230.6, 193.3)
- added R442: 82, Resistor_SMD:R_0402_1005Metric, B.Cu at (232.6, 192.8)
- added R443: 130, Resistor_SMD:R_0402_1005Metric, B.Cu at (230.6, 192.3)
- added R444: 360, Resistor_SMD:R_0402_1005Metric, B.Cu at (232.6, 191.8)
- added R445: 82, Resistor_SMD:R_0402_1005Metric, B.Cu at (230.6, 191.0)
- added R446: 130, Resistor_SMD:R_0402_1005Metric, B.Cu at (232.6, 190.5)
- added R447: 360, Resistor_SMD:R_0402_1005Metric, B.Cu at (230.6, 190.0)
- added R448: 82, Resistor_SMD:R_0402_1005Metric, B.Cu at (232.6, 189.5)
- added R449: 130, Resistor_SMD:R_0402_1005Metric, B.Cu at (230.6, 188.7)
- added R450: 360, Resistor_SMD:R_0402_1005Metric, B.Cu at (232.6, 188.2)
- added R451: 82, Resistor_SMD:R_0402_1005Metric, B.Cu at (230.6, 187.7)
- added R452: 130, Resistor_SMD:R_0402_1005Metric, B.Cu at (232.6, 187.2)
- added R453: 360, Resistor_SMD:R_0402_1005Metric, B.Cu at (230.6, 186.3)
- added R454: 82, Resistor_SMD:R_0402_1005Metric, B.Cu at (232.6, 185.8)
- added R455: 130, Resistor_SMD:R_0402_1005Metric, B.Cu at (230.6, 185.3)
- added R456: 360, Resistor_SMD:R_0402_1005Metric, B.Cu at (232.6, 184.8)
- added R457: 82, Resistor_SMD:R_0402_1005Metric, B.Cu at (230.6, 184.0)
- added R458: 130, Resistor_SMD:R_0402_1005Metric, B.Cu at (232.6, 183.5)
- added R459: 360, Resistor_SMD:R_0402_1005Metric, B.Cu at (230.6, 183.0)
- added R460: 82, Resistor_SMD:R_0402_1005Metric, B.Cu at (232.6, 182.5)
- added R461: 130, Resistor_SMD:R_0402_1005Metric, B.Cu at (230.6, 181.7)
- added R462: 360, Resistor_SMD:R_0402_1005Metric, B.Cu at (232.6, 181.2)
- added R463: 82, Resistor_SMD:R_0402_1005Metric, B.Cu at (230.6, 180.7)
- added R464: 130, Resistor_SMD:R_0402_1005Metric, B.Cu at (232.6, 180.2)
- added R465: 360, Resistor_SMD:R_0402_1005Metric, B.Cu at (230.6, 179.4)
- added R466: 82, Resistor_SMD:R_0402_1005Metric, B.Cu at (232.6, 178.9)
- added R467: 130, Resistor_SMD:R_0402_1005Metric, B.Cu at (230.6, 178.4)
- added R468: 360, Resistor_SMD:R_0402_1005Metric, B.Cu at (232.6, 177.9)
- added R469: 82, Resistor_SMD:R_0402_1005Metric, B.Cu at (230.6, 177.1)
- added R470: 130, Resistor_SMD:R_0402_1005Metric, B.Cu at (232.6, 176.6)
- added R471: 360, Resistor_SMD:R_0402_1005Metric, B.Cu at (230.6, 176.1)
- added R472: 82, Resistor_SMD:R_0402_1005Metric, B.Cu at (232.6, 175.6)
- added R473: 130, Resistor_SMD:R_0402_1005Metric, B.Cu at (230.6, 174.7)
- added R474: 360, Resistor_SMD:R_0402_1005Metric, B.Cu at (232.6, 174.2)
- added R475: 82, Resistor_SMD:R_0402_1005Metric, B.Cu at (230.6, 173.7)
- added R476: 130, Resistor_SMD:R_0402_1005Metric, B.Cu at (232.6, 173.2)
- added R477: 360, Resistor_SMD:R_0402_1005Metric, B.Cu at (230.6, 172.4)
- added R478: 82, Resistor_SMD:R_0402_1005Metric, B.Cu at (232.6, 171.9)
- added R479: 130, Resistor_SMD:R_0402_1005Metric, B.Cu at (230.6, 171.4)
- added R480: 360, Resistor_SMD:R_0402_1005Metric, B.Cu at (232.6, 170.9)
- added R481: 82, Resistor_SMD:R_0402_1005Metric, B.Cu at (230.6, 170.1)
- added R482: 130, Resistor_SMD:R_0402_1005Metric, B.Cu at (232.6, 169.6)
- added R483: 360, Resistor_SMD:R_0402_1005Metric, B.Cu at (230.6, 169.1)
- added R484: 82, Resistor_SMD:R_0402_1005Metric, B.Cu at (232.6, 168.6)
- added R485: 130, Resistor_SMD:R_0402_1005Metric, B.Cu at (230.6, 167.8)
- added R486: 360, Resistor_SMD:R_0402_1005Metric, B.Cu at (232.6, 167.3)
- added R487: 82, Resistor_SMD:R_0402_1005Metric, B.Cu at (230.6, 166.8)
- added R488: 130, Resistor_SMD:R_0402_1005Metric, B.Cu at (232.6, 166.3)
- added R489: 360, Resistor_SMD:R_0402_1005Metric, B.Cu at (230.6, 165.5)
- added R490: 82, Resistor_SMD:R_0402_1005Metric, B.Cu at (232.6, 165.0)
- added R491: 130, Resistor_SMD:R_0402_1005Metric, B.Cu at (230.6, 164.5)
- added R492: 360, Resistor_SMD:R_0402_1005Metric, B.Cu at (232.6, 164.0)
- added R496: 82, Resistor_SMD:R_0402_1005Metric, B.Cu at (232.6, 161.6)
- added R497: 1k, Resistor_SMD:R_0402_1005Metric, B.Cu at (244.0, 162.3)
- added R498: 1k, Resistor_SMD:R_0402_1005Metric, B.Cu at (244.1, 163.9)
- added R499: 1k, Resistor_SMD:R_0402_1005Metric, B.Cu at (244.0, 165.8)
- added R500: 1k, Resistor_SMD:R_0402_1005Metric, B.Cu at (244.1, 167.4)
- added R501: 1k, Resistor_SMD:R_0402_1005Metric, B.Cu at (244.0, 169.3)
- added R502: 1k, Resistor_SMD:R_0402_1005Metric, B.Cu at (244.1, 170.9)
- added R503: 1k, Resistor_SMD:R_0402_1005Metric, B.Cu at (244.0, 172.8)
- added R504: 1k, Resistor_SMD:R_0402_1005Metric, B.Cu at (244.1, 174.4)
- added R505: 1k, Resistor_SMD:R_0402_1005Metric, B.Cu at (244.0, 176.3)
- added R506: 1k, Resistor_SMD:R_0402_1005Metric, B.Cu at (244.1, 177.9)
- added R507: 1k, Resistor_SMD:R_0402_1005Metric, B.Cu at (244.0, 179.8)
- added R508: 1k, Resistor_SMD:R_0402_1005Metric, B.Cu at (244.1, 181.4)
- added R509: 1k, Resistor_SMD:R_0402_1005Metric, B.Cu at (244.0, 183.3)
- added R510: 1k, Resistor_SMD:R_0402_1005Metric, B.Cu at (244.1, 184.9)
- added R511: 1k, Resistor_SMD:R_0402_1005Metric, B.Cu at (244.0, 186.8)
- added R512: 1k, Resistor_SMD:R_0402_1005Metric, B.Cu at (244.1, 188.4)
- added R513: 1k, Resistor_SMD:R_0402_1005Metric, B.Cu at (244.0, 190.3)
- added R514: 1k, Resistor_SMD:R_0402_1005Metric, B.Cu at (244.1, 191.9)
- added R515: 1k, Resistor_SMD:R_0402_1005Metric, B.Cu at (244.0, 193.8)
- added R516: 1k, Resistor_SMD:R_0402_1005Metric, B.Cu at (244.1, 195.4)
- added R517: 1k, Resistor_SMD:R_0402_1005Metric, B.Cu at (244.0, 197.3)
- added R518: 1k, Resistor_SMD:R_0402_1005Metric, B.Cu at (244.1, 198.9)
- added R519: 1k, Resistor_SMD:R_0402_1005Metric, B.Cu at (244.0, 200.8)
- added R520: 1k, Resistor_SMD:R_0402_1005Metric, B.Cu at (244.1, 202.4)
- added R521: 1k, Resistor_SMD:R_0402_1005Metric, B.Cu at (244.0, 204.3)
- added R522: 1k, Resistor_SMD:R_0402_1005Metric, B.Cu at (244.1, 205.9)
- added R523: 1k, Resistor_SMD:R_0402_1005Metric, B.Cu at (244.0, 207.8)
- added R524: 1k, Resistor_SMD:R_0402_1005Metric, B.Cu at (244.1, 209.4)
- added R525: 1k, Resistor_SMD:R_0402_1005Metric, B.Cu at (244.0, 211.3)
- added R526: 1k, Resistor_SMD:R_0402_1005Metric, B.Cu at (244.1, 212.9)
- added R527: 1k, Resistor_SMD:R_0402_1005Metric, B.Cu at (244.0, 214.8)
- added R528: 1k, Resistor_SMD:R_0402_1005Metric, B.Cu at (244.1, 216.4)
- added U401: 74HC595BQ, Package_DFN_QFN:DHVQFN-16-1EP_2.5x3.5mm_P0.5mm_EP1x2mm, B.Cu at (235.7, 214.4)
- added U402: 74HC595BQ, Package_DFN_QFN:DHVQFN-16-1EP_2.5x3.5mm_P0.5mm_EP1x2mm, B.Cu at (235.7, 209.7)
- added U403: 74HC595BQ, Package_DFN_QFN:DHVQFN-16-1EP_2.5x3.5mm_P0.5mm_EP1x2mm, B.Cu at (235.7, 205.1)
- added U404: 74HC595BQ, Package_DFN_QFN:DHVQFN-16-1EP_2.5x3.5mm_P0.5mm_EP1x2mm, B.Cu at (235.7, 200.4)
- added U405: 74HC595BQ, Package_DFN_QFN:DHVQFN-16-1EP_2.5x3.5mm_P0.5mm_EP1x2mm, B.Cu at (235.7, 195.8)
- added U406: 74HC595BQ, Package_DFN_QFN:DHVQFN-16-1EP_2.5x3.5mm_P0.5mm_EP1x2mm, B.Cu at (235.7, 191.2)
- added U407: 74HC595BQ, Package_DFN_QFN:DHVQFN-16-1EP_2.5x3.5mm_P0.5mm_EP1x2mm, B.Cu at (235.7, 186.5)
- added U408: 74HC595BQ, Package_DFN_QFN:DHVQFN-16-1EP_2.5x3.5mm_P0.5mm_EP1x2mm, B.Cu at (235.7, 181.9)
- added U409: 74HC595BQ, Package_DFN_QFN:DHVQFN-16-1EP_2.5x3.5mm_P0.5mm_EP1x2mm, B.Cu at (235.7, 177.2)
- added U410: 74HC595BQ, Package_DFN_QFN:DHVQFN-16-1EP_2.5x3.5mm_P0.5mm_EP1x2mm, B.Cu at (235.7, 172.6)
- added U411: 74HC595BQ, Package_DFN_QFN:DHVQFN-16-1EP_2.5x3.5mm_P0.5mm_EP1x2mm, B.Cu at (235.7, 168.0)
- added U413: 74HC138LQ/TR, Package_DFN_QFN:QFN-16-1EP_3x3mm_P0.5mm_EP1.7x1.7mm_ThermalVias, B.Cu at (247.2, 168.5)
- added U414: 74HC138LQ/TR, Package_DFN_QFN:QFN-16-1EP_3x3mm_P0.5mm_EP1.7x1.7mm_ThermalVias, B.Cu at (248.2, 188.9)
- added U415: 74HC138LQ/TR, Package_DFN_QFN:QFN-16-1EP_3x3mm_P0.5mm_EP1.7x1.7mm_ThermalVias, B.Cu at (247.2, 182.5)
- added U416: 74HC138LQ/TR, Package_DFN_QFN:QFN-16-1EP_3x3mm_P0.5mm_EP1.7x1.7mm_ThermalVias, B.Cu at (247.2, 196.5)
- added U417: 74HC138LQ/TR, Package_DFN_QFN:QFN-16-1EP_3x3mm_P0.5mm_EP1.7x1.7mm_ThermalVias, B.Cu at (247.2, 210.5)
- R493: renamed from R67; value 130 -> 82
- R494: renamed from R68; value 360 -> 130
- R495: renamed from R69; value 82 -> 360
- moved C402 139.1 mm to (303.3, 202.6), turned to -90 degrees
- moved U412 136.9 mm to (235.7, 163.3), turned to 0 degrees
- moved R495 115.3 mm to (230.6, 162.1)
- moved U418 113.6 mm to (254.2, 193.9), turned to 0 degrees
- moved R494 113.0 mm to (232.6, 162.6)
- moved R493 110.4 mm to (230.6, 163.1)
- moved D1 54.3 mm to (173.9, 216.2), turned to -90 degrees
- moved D10 54.3 mm to (189.7, 216.2), turned to -90 degrees
- moved D11 54.3 mm to (191.4, 216.2), turned to -90 degrees
- moved D12 54.3 mm to (193.2, 216.2), turned to -90 degrees
- moved D13 54.3 mm to (194.9, 216.2), turned to -90 degrees
- moved D14 54.3 mm to (196.7, 216.2), turned to -90 degrees
- moved D15 54.3 mm to (198.4, 216.2), turned to -90 degrees
- moved D16 54.3 mm to (200.2, 216.2), turned to -90 degrees
- moved D17 54.3 mm to (201.9, 216.2), turned to -90 degrees
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- renumbered AE2 to AE601, AE1 to AE602, BT1 to BT301, BZ1 to BZ101, C43 to C101, C45 to C102, C46 to C103, C47 to C104, C49 to C105, C50 to C106, C51 to C107, C52 to C108, C53 to C109, C54 to C110, C55 to C111, C56 to C112, C48 to C113, C44 to C114, C41 to C115, C42 to C116, C3 to C117, C40 to C118, C6 to C201, C8 to C202, C9 to C203, C10 to C204, C12 to C205, C13 to C206, C14 to C207, C15 to C208, C16 to C209, C17 to C210, C18 to C211, C39 to C212, C11 to C213, C7 to C214, C4 to C215, C5 to C216, C1 to C217, C2 to C218, C57 to C301, C61 to C302, C62 to C303, C58 to C304, C60 to C305, C63 to C306, C64 to C307, C59 to C308, C26 to C401, C27 to C402, C28 to C403, C29 to C404, C30 to C405, C31 to C406, C32 to C407, C33 to C408, C34 to C409, C69 to C601, C70 to C602, C71 to C603, C72 to C604, C73 to C605, C74 to C606, C77 to C607, C78 to C608, C79 to C609, C20 to C610, C68 to C611, C80 to C612, C75 to C613, C76 to C614, C81 to C615, C89 to C616, C84 to C617, C86 to C618, C90 to C619, C91 to C620, C85 to C621, C87 to C622, C88 to C623, C82 to C624, C83 to C625, C19 to C626, C65 to C627, C67 to C628, C66 to C629, J6 to J101, J1 to J102, J5 to J201, J7 to J202, J3 to J301, L3 to L101, L1 to L201, L2 to L301, L6 to L601, L7 to L602, L4 to L603, L5 to L604, Q21 to Q201, Q22 to Q301, Q23 to Q302, R50 to R101, R51 to R102, R52 to R103, R49 to R104, R41 to R105, R47 to R106, R48 to R107, R5 to R201, R7 to R202, R8 to R203, R3 to R204, R2 to R205, R54 to R206, R53 to R207, R42 to R208, R56 to R301, R55 to R302, R59 to R303, R63 to R304, R62 to R305, R64 to R306, R60 to R307, R61 to R308, R66 to R309, R65 to R310, R4 to R601, R6 to R602, SW1 to SW101, SW2 to SW102, SW7 to SW201, SW4 to SW202, SW3 to SW301, TP19 to TP101, TP16 to TP201, TP1 to TP202, TP2 to TP203, TP3 to TP204, TP4 to TP205, TP18 to TP301, TP12 to TP302, TP17 to TP303, TP13 to TP304, TP14 to TP305, TP5 to TP601, TP6 to TP602, U23 to U101, U30 to U201, U24 to U301, U19 to U302, U1 to U412, U18 to U418, U21 to U601, U20 to U602, VCC1 to VCC601, VCC3 to VCC602, VCC2 to VCC603, Y2 to Y101, Y1 to Y201, Y4 to Y601, Y3 to Y602
Connections:
- AE602 pad : (no net) -> GND
- R493 pad 1: Net-(U1-QA) -> Net-(U412-QE)
- R493 pad 2: /LED_control/LED_matrix/R0 -> /LED_control/LED_matrix/B30
- R494 pad 1: Net-(U1-QB) -> Net-(U412-QF)
- R494 pad 2: /LED_control/LED_matrix/G0 -> /LED_control/LED_matrix/R31
- R495 pad 1: Net-(U1-QC) -> Net-(U412-QG)
- R495 pad 2: /LED_control/LED_matrix/B0 -> /LED_control/LED_matrix/G31
- U101 pad 49: unconnected-(U23-GPIO40_ADC0-Pad49) -> Net-(U101-GPIO40_ADC0)
- U101 pad 52: unconnected-(U23-GPIO41_ADC1-Pad52) -> Net-(U101-GPIO41_ADC1)
- U101 pad 53: unconnected-(U23-GPIO42_ADC2-Pad53) -> Net-(U101-GPIO42_ADC2)
- U101 pad 54: unconnected-(U23-GPIO43_ADC3-Pad54) -> Net-(U101-GPIO43_ADC3)
- U412 pad 1: Net-(U1-QB) -> Net-(U412-QB)
- U412 pad 14: /Display_Unit/DISP-R_S_1 -> /Display_Unit/DISP-R_S_12
- U412 pad 15: Net-(U1-QA) -> Net-(U412-QA)
- U412 pad 2: Net-(U1-QC) -> Net-(U412-QC)
- U412 pad 4: Net-(U1-QE) -> Net-(U412-QE)
- U412 pad 5: Net-(U1-QF) -> Net-(U412-QF)
- U412 pad 6: Net-(U1-QG) -> Net-(U412-QG)
- U602 pad 17: (no net) -> GND
Routing:
- net +3V3: track 112.3 -> 426.4 mm, vias 55 -> 117
- net /Display_Unit/DISP-R_S_1: track 3.47 -> 85.1 mm, vias 0 -> 2
- net /Display_Unit/DISP-R_S_2: track 1.73 -> 81.2 mm, vias 0 -> 2
- net /Display_Unit/DISP-STOP: track 38.8 -> 116.7 mm, vias 3 -> 13
- net /Display_Unit/DISP-C_P_1: track 18.0 -> 87.8 mm, vias 1 -> 7
- net /Display_Unit/DISP-C_P_3: track 16.9 -> 86.0 mm, vias 1 -> 7
- net /Display_Unit/DISP-C_P_2: track 19.7 -> 86.6 mm, vias 1 -> 6
- net /Display_Unit/DISP-R_S_5: track 2.75 -> 69.6 mm, vias 0 -> 2
- net /Display_Unit/DISP-~{OE}: track 39.6 -> 106.1 mm, vias 3 -> 13
- net /Display_Unit/DISP-R_S_6: track 4.26 -> 69.3 mm, vias 0 -> 2
- net /Display_Unit/DISP-R_S_7: track 1.10 -> 66.1 mm, vias 1 -> 2
- net /Display_Unit/DISP-CLK: track 38.1 -> 99.8 mm, vias 3 -> 13
- net /Display_Unit/DISP-R_S_8: track 4.13 -> 61.3 mm, vias 0 -> 2
- net /Display_Unit/DISP-R_S_9: track 4.39 -> 59.7 mm, vias 0 -> 2
- net /Display_Unit/DISP-R_S_10: track 4.38 -> 56.0 mm, vias 0 -> 2
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Other:
- board text removed: "BOOT"
- board text removed: "U13"
