File: hardware/full-poc/rf.kicad_sch (KiCad schematic)
At the start: 46 parts, among them U20 CMT2219A, U21 ST25R3916B-AQWT, Y3 TAXM26M4RHBCCT2T, Y4 5YMA27120091KF50EB

Commit message: full board + panel
Parts:
- renumbered AE2 to AE601, AE1 to AE602, C69 to C601, C70 to C602, C71 to C603, C72 to C604, C73 to C605, C74 to C606, C77 to C607, C78 to C608, C79 to C609, C20 to C610, C68 to C611, C80 to C612, C75 to C613, C76 to C614, C81 to C615, C89 to C616, C84 to C617, C86 to C618, C90 to C619, C91 to C620, C85 to C621, C87 to C622, C88 to C623, C82 to C624, C83 to C625, C19 to C626, C65 to C627, C67 to C628, C66 to C629, L6 to L601, L7 to L602, L4 to L603, L5 to L604, R4 to R601, R6 to R602, TP5 to TP601, TP6 to TP602, U21 to U601, U20 to U602, VCC1 to VCC601, VCC3 to VCC602, VCC2 to VCC603, Y4 to Y601, Y3 to Y602
